File: hardware/v1.0/QMTECH_XC7A100T-Expantion-Board.kicad_sch (KiCad schematic)
At the start: 29 parts, among them J1 Micro_SD_Card_Det1, J14 USB_C_Receptacle_USB2.0_16P, J15 Conn_02x06_Top_Bottom, J16 Conn_02x06_Top_Bottom, J2 Conn_01x34, J3 USB_C_Receptacle_USB2.0_16P, J4 Conn_01x34, Q1 AON6411, U14 HUSB238, U15 CH340C

Commit message: first schematic iteration done
Parts:
- removed J15, J16: Conn_02x06_Top_Bottom, Connector_PinSocket_2.54mm:PinSocket_2x06_P2.54mm_Horizontal, symbol Connector_Generic:Conn_02x06_Top_Bottom
- removed U15: CH340C, Package_SO:SOIC-16_3.9x9.9mm_P1.27mm, symbol Interface_USB:CH340C
- added C22, C24: 1nf 2kv, symbol Device:C_Small
- added C23: 0.1uf, symbol Device:C_Small
- added D10, D11, D3, D5, D6, D7, D8, D9: ~, LED_SMD:LED_0805_2012Metric, symbol Device:LED_Small
- added D12: ~, C779813:LED-SMD_4P-L1.6-W1.5-BR_TZ-P4-1615, symbol Device:LED_ARGB
- added J15, J16: Conn_02x06_Odd_Even, Connector_PinSocket_2.54mm:PinSocket_2x06_P2.54mm_Horizontal, symbol Connector_Generic:Conn_02x06_Odd_Even
- added R28: 4.7k, Resistor_SMD:R_0603_1608Metric_Pad0.98x0.95mm_HandSolder, symbol Device:R_Small
- added R40, R41: 1m, symbol Device:R_Small
- added RN21, RN24, RN25, RN26, RN27: 5.1k, symbol Device:R_Pack02
- added U15: CH340C, Package_SO:SOIC-16_3.9x9.9mm_P1.27mm, symbol mylib:CH340C
- U16, U3: footprint (none) -> Package_DFN_QFN:Diodes_UDFN-10_1.0x2.5mm_P0.5mm
Connections:
- net +3V3: now also C23.1, J15.11 (Pin_11), J15.12 (Pin_12), J16.11 (Pin_11), J16.12 (Pin_12), R28.2, U15.16 (VCC), U15.4 (V3)
- net GND: now also J14.A1 (GND), J14.A12 (GND), J14.B1 (GND), J14.B12 (GND), U16.3 (VSS), U16.8 (VSS), C22.2, C23.2, C24.1, D12.2 (RK), J15.10 (Pin_10), J15.9 (Pin_9), J16.10 (Pin_10), J16.9 (Pin_9), R40.2, R41.1, RN21.3 (R2.2), RN21.4 (R1.2), RN24.1 (R1.1), RN24.2 (R2.1), RN25.1 (R1.1), RN25.2 (R2.1), RN26.1 (R1.1), RN26.2 (R2.1), RN27.1 (R1.1), RN27.2 (R2.1), U15.1 (GND); no longer J3.S1 (SHIELD)
- net at J14.A5 (CC1): now also RN21.2 (R2.1)
- net UART_DP: now reaches J14.A6 (D+)
- net UART_DP: now also J14.B6 (D+), U16.2, U16.9 (NC), U15.5 (UD+)
- net UART_DN: now reaches J14.A7 (D-)
- net UART_DN: now also J14.B7 (D-), U16.1, U16.10 (NC), U15.6 (UD-)
- net at J14.B5 (CC2): now also RN21.1 (R1.1)
- net at J14.S1 (SHIELD): now also C22.1, R40.1
- net at U16.4: now also U16.7 (NC)
- net at U16.5: now also U16.6 (NC)
- net PMOD1_3P: now reaches U1.71 (IO_B5)
- net PMOD1_3P: now also J16.7 (Pin_7)
- net PMOD1_3N: now reaches U1.72 (IO_A5)
- net PMOD1_3N: now also J16.8 (Pin_8)
- net PMOD1_2P: now reaches U1.73 (IO_B4)
- net PMOD1_2P: now also J16.5 (Pin_5)
- net PMOD1_2N: now reaches U1.74 (IO_A4)
- net PMOD1_2N: now also J16.6 (Pin_6)
- net PMOD1_1P: now reaches U1.75 (IO_A3)
- net PMOD1_1P: now also J16.3 (Pin_3)
- net PMOD1_1N: now reaches U1.76 (IO_A2)
- net PMOD1_1N: now also J16.4 (Pin_4)
- net PMOD1_0P: now reaches U1.77 (IO_D4)
- net PMOD1_0P: now also J16.1 (Pin_1)
- net PMOD1_0N: now reaches U1.78 (IO_C4)
- net PMOD1_0N: now also J16.2 (Pin_2)
- net PMOD0_3P: now reaches U1.79 (IO_C2)
- net PMOD0_3P: now also J15.7 (Pin_7)
- net PMOD0_3N: now reaches U1.80 (IO_B2_VREF)
- net PMOD0_3N: now also J15.8 (Pin_8)
- net PMOD0_2P: now reaches U1.81 (IO_E5)
- net PMOD0_2P: now also J15.5 (Pin_5)
- net PMOD0_2N: now reaches U1.82 (IO_D5)
- net PMOD0_2N: now also J15.6 (Pin_6)
- net PMOD0_1P: now reaches U1.83 (IO_C1)
- net PMOD0_1P: now also J15.3 (Pin_3)
- net PMOD0_1N: now reaches U1.84 (IO_B1)
- net PMOD0_1N: now also J15.4 (Pin_4)
- net PMOD0_0P: now reaches U1.85 (IO_E1)
- net PMOD0_0P: now also J15.1 (Pin_1)
- net PMOD0_0N: now reaches U1.86 (IO_D1)
- net PMOD0_0N: now also J15.2 (Pin_2)
- net STATUS1: now reaches U1.95 (IO_H2)
- net STATUS1: now also D12.3 (GK)
- net STATUS0: now reaches U1.96 (IO_H1)
- net STATUS0: now also D12.4 (BK)
- new net: D5.1 (K), RN24.4 (R1.2)
- new net: D7.1 (K), RN25.4 (R1.2)
- new net: D12.1 (A), R28.1
- new net: D8.1 (K), RN26.3 (R2.2)
- new net: D10.1 (K), RN27.3 (R2.2)
- new net: D11.1 (K), RN27.4 (R1.2)
- new net: C24.2, J3.S1 (SHIELD), R41.2
- new net: D6.1 (K), RN25.3 (R2.2)
- new net: D9.1 (K), RN26.4 (R1.2)
- new net: D3.1 (K), RN24.3 (R2.2)
- new net LED0_0: D8.2 (A)
- new net LED0_1: D9.2 (A)
- new net LED0_2: D10.2 (A)
- new net LED0_3: D11.2 (A)
- new net LED0_4: D3.2 (A)
- new net LED0_5: D5.2 (A)
- new net LED0_6: D6.2 (A)
- new net LED0_7: D7.2 (A)
- new net UART_RX: U15.3 (RXD)
- new net UART_TX: U15.2 (TXD)
- no-connect marks 4 -> 14
Other:
- note added: "INDICATOR"
- note added: "UART"
- moved on the sheet: J1, J14, J2, R1, R2, R3, R4, R5, R6, R7, U16, U1A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
